File: svarog-keyboard.sch (KiCad schematic (older format))
At the start: 250 parts, among them J1 USB_mini_micro_B, K1 KEYSW, K10 KEYSW, K11 KEYSW, K12 KEYSW, K13 KEYSW, K14 KEYSW, K15 KEYSW, K16 KEYSW, K17 KEYSW, K18 KEYSW, K19 KEYSW, K2 KEYSW, K20 KEYSW, K21 KEYSW, K3 KEYSW, K4 KEYSW, K5 KEYSW, K6 KEYSW, K7 KEYSW, K8 KEYSW, K9 KEYSW, SW1 SW_PUSH, U1 ATMEGA32U4, X1 XTAL_GND

Commit message: Added I/O expander
Parts:
- added C9: 4.7u, symbol Device:C_Small
- added D14-1, D14-2: D, symbol Device:D
- added K13-1, K14-1, K14-2, K_Ent-1, K_LS-1, K_R16-1: KEYSW, symbol keyboard_parts:KEYSW
- added U2: MCP23017_SO, Package_SO:SOIC-28W_7.5x17.9mm_P1.27mm, symbol Interface_Expansion:MCP23017_SO
Connections:
- net GND: now also C9.2, U2.10 (VSS)
- net SCK: now also U2.12 (SCK)
- net VCC: now also C9.1, U2.18 (~RESET~), U2.9 (VDD)
- net col_1: now also D14-2.1 (K)
- net col_10: now also K6.1, KB.1, KH.1, KY.1
- net col_11: now also K7.1, KJ.1, KN.1, KU.1, K_SPC.1
- net col_12: now also K8.1, KI.1, KK.1, KM.1
- net col_13: now also K19.1, K9.1, KL.1, KO.1
- net col_14: now also K10.1, K17.1, K20.1, KP.1
- net col_15: now also K11.1, K15.1, K18.1, K21.1, K_RA.1
- net col_16: now also K12.1, K16.1, K_Fn.1
- net col_17: now also K13.1, K_Men.1, K13-1.1, K14-1.1
- net col_18: now also K14.1, K_Bsc.1, K_Ent.1, K_RC.1, K_RS.1, K_Ent-1.1
- net col_19: now also K_R16-1.1
- net col_4: now also K_CL.1, K_Esc.1, K_LC.1, K_LS.1, K_Tb.1, K_LS-1.1
- net col_5: now also K1.1, KA.1, KQ.1, K_LSu.1, K14-2.1
- net col_6: now also K2.1, KS.1, KW.1, KZ.1, K_LA.1
- net col_7: now also K3.1, KD.1, KE.1, KX.1
- net col_8: now also K4.1, KC.1, KF.1, KR.1
- net col_9: now also K5.1, KG.1, KT.1, KV.1
- net col_f0: now also U2.3 (GPB2)
- net col_f1: now also U2.4 (GPB3)
- net col_f10: now also U2.25 (GPA4)
- net col_f11: now also U2.26 (GPA5)
- net col_f2: now also U2.5 (GPB4)
- net col_f3: now also U2.6 (GPB5)
- net col_f4: now also U2.7 (GPB6)
- net col_f5: now also U2.8 (GPB7)
- net col_f6: now also U2.21 (GPA0)
- net col_f7: now also U2.22 (GPA1)
- net col_f8: now also U2.23 (GPA2)
- net col_f9: now also U2.24 (GPA3)
- net row_3: now also D14-1.1 (K)
- net row_f0: now also U2.1 (GPB0)
- net row_f1: now also U2.2 (GPB1)
- net at D_LS.2 (A), K_LS.2: now also K_LS-1.2
- net at D_R16.2 (A), K_R16.2: now also K_R16-1.2
- net at D13.2 (A), K13.2: now also K13-1.2
- net at D_Ent.2 (A), K_Ent.2: now also K_Ent-1.2
- net MISO: no longer names the net of U1.11 (PB3/MISO)
- net MOSI: no longer names the net of U1.10 (PB2/MOSI)
- net RTS: no longer names the net of U1.12 (PB7/~RTS)
- net SS renamed SDA
- net SDA: now also U2.13 (SDA)
- new net: D14-2.2 (A), K14-2.2
- new net: D14-1.2 (A), K14-1.2
- no-connect marks 18 -> 28
Other:
- note added: "Alphas (Switch Matrix)"
- note added: "Function Row (Switch Matrix)\n"
- note added: "I/O Expander"
- note added: "Navigation (Switch Matrix)\n"
- note added: "Numerical (Switch Matrix)"
- moved on the sheet: C1, C2, C3, C4, C5, C6, C7, C8, D1, D10, D11, D12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

Commit message: Changed MCU from 32U4 to 32A, added new I/O expanders
Parts:
- removed C1, C2: 22p, symbol Device:C_Small
- removed C3, C4, C5, C6: 0.1u, symbol Device:C_Small
- removed J1: USB_mini_micro_B, symbol keyboard_parts:USB_mini_micro_B
- removed SW1: SW_PUSH, symbol keyboard_parts:SW_PUSH
- removed U1: ATMEGA32U4, symbol keyboard_parts:ATMEGA32U4
- removed X1: XTAL_GND, symbol keyboard_parts:XTAL_GND
- added C1, C2: 22p, symbol Device:C
- added C3: 4.7u, symbol Device:CP1
- added C4, C5: 0.1u, symbol Device:C
- added DZ1, DZ2: 3.6V, symbol Device:D_Zener
- added F1: 500mA, symbol Device:Polyfuse
- added J1: AVR-ISP-6, symbol Connector:AVR-ISP-6
- added J2: USB_C_Receptacle, symbol Connector:USB_C_Receptacle
- added LED, LED2, LED3, LED4: POWER, symbol Device:LED
- added R10, R5, R8, R9: 1.5k, symbol Device:R
- added R6, R7: 5.1k, symbol Device:R
- added SW1: SW_BOOT, symbol Switch:SW_Push
- added SW2: SW_RESET, symbol Switch:SW_Push
- added U1: ATmega32A-PU, Package_DIP:DIP-40_W15.24mm, symbol MCU_Microchip_ATmega:ATmega32A-PU
- added U3, U4: MCP23017_SO, Package_SO:SOIC-28W_7.5x17.9mm_P1.27mm, symbol Interface_Expansion:MCP23017_SO
- added Y1: Crystal, symbol Device:Crystal
- C8: value 1u -> 4.7u
- R2: value 10k -> 1.5k
- R3, R4: value 22 -> 75R
- renumbered C9 to C6
Connections:
- net col_16 is gone; now on net col_13: K12.1, K16.1, K_Fn.1
- net col_17 is gone; now on net col_14: K13-1.1, K13.1, K14-1.1, K_Men.1
- net col_18 is gone; now on net col_15: K14.1, K_Bsc.1, K_Ent-1.1, K_Ent.1, K_RC.1, K_RS.1
- net GND: now also R2.2, U2.15 (A0), C1.2, C2.2, C3.2, C4.2, C5.2, DZ1.2 (A), DZ2.2 (A), J1.6 (GND), J2.A1 (GND), J2.A12 (GND), J2.B1 (GND), J2.B12 (GND), J2.S1 (SHIELD), R10.2, R6.1, R7.1, R8.2, R9.2, SW1.1, SW2.1, U3.10 (VSS), U3.16 (A1), U4.10 (VSS), U4.15 (A0), U4.16 (A1); no longer R2.1
- net SCK: now also J1.3 (SCK), U1.8 (PB7); no longer U2.12 (SCK)
- net VCC: now also C8.1, F1.2, J2.A4 (VBUS), J2.A9 (VBUS), J2.B4 (VBUS), J2.B9 (VBUS); no longer R1.2, U2.18 (~RESET~), U2.9 (VDD)
- net col_1: now also K_CL.1, K_Esc.1, K_LC.1, K_LS-1.1, K_LS.1, K_Tb.1, U1.38 (PA2); no longer D14-2.1 (K), D19.1 (K), D20.1 (K), D21.1 (K), DB.1 (K), DC.1 (K), DM.1 (K), DN.1 (K), DV.1 (K), DX.1 (K), DZ.1 (K), D_L13.1 (K), D_LS.1 (K), D_R12.1 (K), D_R13.1 (K), D_R14.1 (K), D_R15.1 (K), D_RS.1 (K), K_L10.1, K_L14.1, K_L4.1, K_L7.1
- net col_10: now also K19.1, K9.1, KL.1, KO.1, U1.26 (PC4); no longer K6.1, KB.1, KH.1, KY.1
- net col_11: now also K10.1, K17.1, K20.1, KP.1, U1.25 (PC3); no longer K7.1, KJ.1, KN.1, KU.1, K_SPC.1
- net col_12: now also K11.1, K15.1, K18.1, K21.1, K_RA.1, U1.24 (PC2); no longer K8.1, KI.1, KK.1, KM.1
- net col_13: now also U1.23 (PC1); no longer K19.1, K9.1, KL.1, KO.1
- net col_14: now also U1.22 (PC0); no longer K10.1, K17.1, K20.1, KP.1
- net col_15: now also U1.21 (PD7); no longer K11.1, K15.1, K18.1, K21.1, K_RA.1
- net col_2: now also K1.1, K14-2.1, KA.1, KQ.1, K_LSu.1, U1.4 (PB3); no longer K_L11.1, K_L13.1, K_L15.1, K_L5.1, K_L8.1
- net col_3: now also K2.1, KS.1, KW.1, KZ.1, K_LA.1, U1.37 (PA3); no longer K_L12.1, K_L16.1, K_L6.1, K_L9.1
- net col_4: now also K3.1, KD.1, KE.1, KX.1, U1.5 (PB4); no longer K_CL.1, K_Esc.1, K_LC.1, K_LS-1.1, K_LS.1, K_Tb.1
- net col_5: now also K4.1, KC.1, KF.1, KR.1, U1.36 (PA4); no longer K1.1, K14-2.1, KA.1, KQ.1, K_LSu.1
- net col_6: now also K5.1, KG.1, KT.1, KV.1, U1.19 (PD5); no longer K2.1, KS.1, KW.1, KZ.1, K_LA.1
- net col_7: now also K6.1, KB.1, KH.1, KY.1, U1.20 (PD6); no longer K3.1, KD.1, KE.1, KX.1
- net col_8: now also K7.1, KJ.1, KN.1, KU.1, K_SPC.1, U1.28 (PC6); no longer K4.1, KC.1, KF.1, KR.1
- net col_9: now also K8.1, KI.1, KK.1, KM.1, U1.27 (PC5); no longer K5.1, KG.1, KT.1, KV.1
- net row_1: now also U1.3 (PB2); no longer D_L4.1 (K), D_L5.1 (K), D_L6.1 (K), D_R1.1 (K), D_R2.1 (K), D_R3.1 (K), D_R4.1 (K)
- net row_2: now also U1.39 (PA1); no longer D_L7.1 (K), D_L8.1 (K), D_L9.1 (K), D_R5.1 (K), D_R6.1 (K), D_R7.1 (K), D_R8.1 (K)
- net row_3: now also U1.2 (PB1); no longer D_L10.1 (K), D_L11.1 (K), D_L12.1 (K), D_R10.1 (K), D_R11.1 (K), D_R9.1 (K)
- net row_5: now also U1.1 (PB0); no longer D_L14.1 (K), D_L15.1 (K), D_L16.1 (K), D_R16.1 (K), D_R17.1 (K), D_R18.1 (K)
- net +5V: now reaches R1.1
- net +5V: now also U2.18 (~RESET~), U2.9 (VDD), C3.1, C4.1, C5.1, F1.1, J1.2 (VCC), LED.2 (A), LED2.2 (A), LED3.2 (A), LED4.2 (A), R5.1, U1.10 (VCC), U1.30 (AVCC), U3.18 (~RESET~), U3.9 (VDD), U4.18 (~RESET~), U4.9 (VDD)
- net at R3.2: now also DZ1.1 (K), J2.A7 (D-), J2.B7 (D-), R5.2
- net at R4.2: now also DZ2.1 (K), J2.A6 (D+), J2.B6 (D+)
- net D-: now reaches R3.1
- net D-: now also U1.17 (PD3)
- net D+: now reaches R4.1
- net D+: now also U1.16 (PD2)
- net SDA renamed SDA_F
- net SDA_F: now also U1.34 (PA6)
- net col_19 renamed col_r1
- net col_r1: now also U4.6 (GPB5)
- net col_20 renamed col_r2
- net col_r2: now also U4.7 (GPB6)
- net col_21 renamed col_r3
- net col_r3: now also U4.8 (GPB7)
- net col_22 renamed col_r4
- net col_r4: now also U4.21 (GPA0)
- new net: U1.11 (GND), U1.31 (GND)
- new net: C2.1, U1.12 (XTAL2), Y1.2
- new net: C1.1, U1.13 (XTAL1), Y1.1
- new net: LED.1 (K), R2.1
- new net: J2.A5 (CC1), R6.2
- new net: J2.B5 (CC2), R7.2
- new net: LED4.1 (K), R10.1
- new net: LED3.1 (K), R9.1
- new net: LED2.1 (K), R8.1
- new net BOOT: SW1.2, U1.18 (PD4)
- new net MISO: J1.1 (MISO), U1.7 (PB6)
- new net MOSI: J1.4 (MOSI), U1.6 (PB5)
- new net RESET: J1.5 (~RST), R1.2, SW2.2, U1.9 (~RESET)
- new net SCK_F: U1.35 (PA5), U2.12 (SCK)
- new net SCK_L: U1.33 (PA7), U3.12 (SCK)
- new net SCK_R: U1.14 (PD0), U4.12 (SCK)
- new net SDA_L: U1.29 (PC7), U3.13 (SDA)
- new net SDA_R: U1.15 (PD1), U4.13 (SDA)
- new net col_l1: D_L13.1 (K), K_L10.1, K_L14.1, K_L4.1, K_L7.1, U3.4 (GPB3), U3.6 (GPB5)
- new net col_l2: K_L11.1, K_L13.1, K_L15.1, K_L5.1, K_L8.1, U3.7 (GPB6)
- new net col_l3: K_L12.1, K_L16.1, K_L6.1, K_L9.1, U3.8 (GPB7)
- new net row_4: D14-2.1 (K), D19.1 (K), D20.1 (K), D21.1 (K), DB.1 (K), DC.1 (K), DM.1 (K), DN.1 (K), DV.1 (K), DX.1 (K), DZ.1 (K), D_LS.1 (K), D_RS.1 (K), U1.40 (PA0)
- new net row_l1: D_L4.1 (K), D_L5.1 (K), D_L6.1 (K), U3.1 (GPB0)
- new net row_l2: D_L7.1 (K), D_L8.1 (K), D_L9.1 (K), U3.2 (GPB1)
- new net row_l3: D_L10.1 (K), D_L11.1 (K), D_L12.1 (K), U3.3 (GPB2)
- new net row_l5: D_L14.1 (K), D_L15.1 (K), D_L16.1 (K), U3.5 (GPB4)
- new net row_r1: D_R1.1 (K), D_R2.1 (K), D_R3.1 (K), D_R4.1 (K), U4.1 (GPB0)
- new net row_r2: D_R5.1 (K), D_R6.1 (K), D_R7.1 (K), D_R8.1 (K), U4.2 (GPB1)
- new net row_r3: D_R10.1 (K), D_R11.1 (K), D_R9.1 (K), U4.3 (GPB2)
- new net row_r4: D_R12.1 (K), D_R13.1 (K), D_R14.1 (K), D_R15.1 (K), U4.4 (GPB3)
- new net row_r5: D_R16.1 (K), D_R17.1 (K), D_R18.1 (K), U4.5 (GPB4)
- no-connect marks 28 -> 39
Other:
- note added: "I/O Expander (F Row)"
- note added: "I/O Expander (Left)"
- note added: "I/O Expander (Right)"
- note added: "MCU and Connector"
- note removed: "I/O Expander"
- moved on the sheet: C6, D_F1, D_F10, D_F11, D_F12, D_F13, D_F14, D_F15, D_F16, D_F17, D_F18, D_F19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

Commit message: Starting adding footprints
Parts:
- removed J2: USB_C_Receptacle, symbol Connector:USB_C_Receptacle
- removed U2, U3, U4: MCP23017_SO, Package_SO:SOIC-28W_7.5x17.9mm_P1.27mm, symbol Interface_Expansion:MCP23017_SO
- added J2: Conn_01x08_Male, Connector_PinHeader_1.00mm:PinHeader_1x08_P1.00mm_Vertical, symbol Connector:Conn_01x08_Male
- added J3, J4, J5, J6: I2C, Connector_PinHeader_1.00mm:PinHeader_1x04_P1.00mm_Vertical, symbol Connector:Conn_01x04_Female
- added LED5: Num Lock, LED_THT:LED_D3.0mm, symbol Device:LED
- added LED6: Scroll Lock, LED_THT:LED_D3.0mm, symbol Device:LED
- added LED7: Caps Lock, LED_THT:LED_D3.0mm, symbol Device:LED
- added R11, R12: 10k, Resistor_THT:R_Axial_DIN0207_L6.3mm_D2.5mm_P7.62mm_Horizontal, symbol Device:R
- added U2, U3, U4: MCP23017_SP, Package_DIP:DIP-28_W7.62mm_Socket, symbol Interface_Expansion:MCP23017_SP
- C3, C6, C7, C8: footprint (none) -> Capacitor_THT:CP_Radial_D4.0mm_P1.50mm
- D1, D10, D11, D12, D13, D14-1, D14-2, D15, D16, D17, D18, D19, D2, D20, D21, D3, D4, D5, D6, D7, D8, D9, D_14, D_F1, D_F10, D_F11, D_F12, D_F13, D_F14, D_F15, D_F16, D_F17, D_F18, D_F19, D_F2, D_F20, D_F21, D_F22, D_F23, D_F24, D_F3, D_F4, D_F5, D_F6, D_F7, D_F8, D_F9, D_L10, D_L11, D_L12, D_L13, D_L14, D_L15, D_L16, D_L4, D_L5, D_L6, D_L7, D_L8, D_L9, D_R1, D_R10, D_R11, D_R12, D_R13, D_R14, D_R15, D_R16, D_R17, D_R18, D_R2, D_R3, D_R4, D_R5, D_R6, D_R7, D_R8, D_R9: footprint (none) -> Diode_THT:D_DO-35_SOD27_P7.62mm_Horizontal
- DA1: renamed from DA; footprint (none) -> Diode_THT:D_DO-35_SOD27_P7.62mm_Horizontal
- DB1: renamed from DB; footprint (none) -> Diode_THT:D_DO-35_SOD27_P7.62mm_Horizontal
- DC1: renamed from DC; footprint (none) -> Diode_THT:D_DO-35_SOD27_P7.62mm_Horizontal
- DD1: renamed from DD; footprint (none) -> Diode_THT:D_DO-35_SOD27_P7.62mm_Horizontal
- DE1: renamed from DE; footprint (none) -> Diode_THT:D_DO-35_SOD27_P7.62mm_Horizontal
- DF1: renamed from DF; footprint (none) -> Diode_THT:D_DO-35_SOD27_P7.62mm_Horizontal
- DG1: renamed from DG; footprint (none) -> Diode_THT:D_DO-35_SOD27_P7.62mm_Horizontal
- DH1: renamed from DH; footprint (none) -> Diode_THT:D_DO-35_SOD27_P7.62mm_Horizontal
- DI1: renamed from DI; footprint (none) -> Diode_THT:D_DO-35_SOD27_P7.62mm_Horizontal
- DJ1: renamed from DJ; footprint (none) -> Diode_THT:D_DO-35_SOD27_P7.62mm_Horizontal
- DK1: renamed from DK; footprint (none) -> Diode_THT:D_DO-35_SOD27_P7.62mm_Horizontal
- DL1: renamed from DL; footprint (none) -> Diode_THT:D_DO-35_SOD27_P7.62mm_Horizontal
- DM1: renamed from DM; footprint (none) -> Diode_THT:D_DO-35_SOD27_P7.62mm_Horizontal
- DN1: renamed from DN; footprint (none) -> Diode_THT:D_DO-35_SOD27_P7.62mm_Horizontal
- DO1: renamed from DO; footprint (none) -> Diode_THT:D_DO-35_SOD27_P7.62mm_Horizontal
- DP1: renamed from DP; footprint (none) -> Diode_THT:D_DO-35_SOD27_P7.62mm_Horizontal
- DQ1: renamed from DQ; footprint (none) -> Diode_THT:D_DO-35_SOD27_P7.62mm_Horizontal
- DR1: renamed from DR; footprint (none) -> Diode_THT:D_DO-35_SOD27_P7.62mm_Horizontal
- DS1: renamed from DS; footprint (none) -> Diode_THT:D_DO-35_SOD27_P7.62mm_Horizontal
- DT1: renamed from DT; footprint (none) -> Diode_THT:D_DO-35_SOD27_P7.62mm_Horizontal
- DU1: renamed from DU; footprint (none) -> Diode_THT:D_DO-35_SOD27_P7.62mm_Horizontal
- DV1: renamed from DV; footprint (none) -> Diode_THT:D_DO-35_SOD27_P7.62mm_Horizontal
- DW1: renamed from DW; footprint (none) -> Diode_THT:D_DO-35_SOD27_P7.62mm_Horizontal
- DX1: renamed from DX; footprint (none) -> Diode_THT:D_DO-35_SOD27_P7.62mm_Horizontal
- DY1: renamed from DY; footprint (none) -> Diode_THT:D_DO-35_SOD27_P7.62mm_Horizontal
- DZ1: renamed from DZ; footprint (none) -> Diode_THT:D_DO-35_SOD27_P7.62mm_Horizontal
- DZ2: renamed from DZ1; footprint (none) -> Diode_THT:D_DO-35_SOD27_P7.62mm_Horizontal
- DZ3: renamed from DZ2; footprint (none) -> Diode_THT:D_DO-35_SOD27_P7.62mm_Horizontal
- D_Bsc1: renamed from D_Bsc; footprint (none) -> Diode_THT:D_DO-35_SOD27_P7.62mm_Horizontal
- D_CL1: renamed from D_CL; footprint (none) -> Diode_THT:D_DO-35_SOD27_P7.62mm_Horizontal
- D_Ent1: renamed from D_Ent; footprint (none) -> Diode_THT:D_DO-35_SOD27_P7.62mm_Horizontal
- D_Esc1: renamed from D_Esc; footprint (none) -> Diode_THT:D_DO-35_SOD27_P7.62mm_Horizontal
- D_Fn1: renamed from D_Fn; footprint (none) -> Diode_THT:D_DO-35_SOD27_P7.62mm_Horizontal
- D_LA1: renamed from D_LA; footprint (none) -> Diode_THT:D_DO-35_SOD27_P7.62mm_Horizontal
- D_LC1: renamed from D_LC; footprint (none) -> Diode_THT:D_DO-35_SOD27_P7.62mm_Horizontal
- D_LS1: renamed from D_LS; footprint (none) -> Diode_THT:D_DO-35_SOD27_P7.62mm_Horizontal
- D_LSu1: renamed from D_LSu; footprint (none) -> Diode_THT:D_DO-35_SOD27_P7.62mm_Horizontal
- D_Men1: renamed from D_Men; footprint (none) -> Diode_THT:D_DO-35_SOD27_P7.62mm_Horizontal
- D_RA1: renamed from D_RA; footprint (none) -> Diode_THT:D_DO-35_SOD27_P7.62mm_Horizontal
- D_RC1: renamed from D_RC; footprint (none) -> Diode_THT:D_DO-35_SOD27_P7.62mm_Horizontal
- D_RS1: renamed from D_RS; footprint (none) -> Diode_THT:D_DO-35_SOD27_P7.62mm_Horizontal
- D_SPC1: renamed from D_SPC; footprint (none) -> Diode_THT:D_DO-35_SOD27_P7.62mm_Horizontal
- D_Tb1: renamed from D_Tb; footprint (none) -> Diode_THT:D_DO-35_SOD27_P7.62mm_Horizontal
- J1: footprint (none) -> Connector_PinHeader_1.00mm:PinHeader_2x03_P1.00mm_Vertical
- K1, K10, K11, K12, K13, K14, K14-1, K14-2, K15, K16, K17, K18, K19, K2, K20, K21, K3, K4, K5, K6, K7, K8, K9, K_F1, K_F10, K_F11, K_F12, K_F13, K_F14, K_F15, K_F16, K_F17, K_F18, K_F19, K_F2, K_F20, K_F21, K_F22, K_F23, K_F24, K_F3, K_F4, K_F5, K_F6, K_F7, K_F8, K_F9: footprint (none) -> Button_Switch_Keyboard:SW_Cherry_MX_1.00u_PCB
- K13-1: footprint (none) -> Button_Switch_Keyboard:SW_Cherry_MX_2.00u_PCB
- KA1: renamed from KA; footprint (none) -> Button_Switch_Keyboard:SW_Cherry_MX_1.00u_PCB
- KB1: renamed from KB; footprint (none) -> Button_Switch_Keyboard:SW_Cherry_MX_1.00u_PCB
- KC1: renamed from KC; footprint (none) -> Button_Switch_Keyboard:SW_Cherry_MX_1.00u_PCB
- KD1: renamed from KD; footprint (none) -> Button_Switch_Keyboard:SW_Cherry_MX_1.00u_PCB
- KE1: renamed from KE; footprint (none) -> Button_Switch_Keyboard:SW_Cherry_MX_1.00u_PCB
- KF1: renamed from KF; footprint (none) -> Button_Switch_Keyboard:SW_Cherry_MX_1.00u_PCB
- KG1: renamed from KG; footprint (none) -> Button_Switch_Keyboard:SW_Cherry_MX_1.00u_PCB
- KH1: renamed from KH; footprint (none) -> Button_Switch_Keyboard:SW_Cherry_MX_1.00u_PCB
- KI1: renamed from KI; footprint (none) -> Button_Switch_Keyboard:SW_Cherry_MX_1.00u_PCB
- KJ1: renamed from KJ; footprint (none) -> Button_Switch_Keyboard:SW_Cherry_MX_1.00u_PCB
- KK1: renamed from KK; footprint (none) -> Button_Switch_Keyboard:SW_Cherry_MX_1.00u_PCB
- KL1: renamed from KL; footprint (none) -> Button_Switch_Keyboard:SW_Cherry_MX_1.00u_PCB
- KM1: renamed from KM; footprint (none) -> Button_Switch_Keyboard:SW_Cherry_MX_1.00u_PCB
- KN1: renamed from KN; footprint (none) -> Button_Switch_Keyboard:SW_Cherry_MX_1.00u_PCB
- KO1: renamed from KO; footprint (none) -> Button_Switch_Keyboard:SW_Cherry_MX_1.00u_PCB
- KP1: renamed from KP; footprint (none) -> Button_Switch_Keyboard:SW_Cherry_MX_1.00u_PCB
- KQ1: renamed from KQ; footprint (none) -> Button_Switch_Keyboard:SW_Cherry_MX_1.00u_PCB
- KR1: renamed from KR; footprint (none) -> Button_Switch_Keyboard:SW_Cherry_MX_1.00u_PCB
- KS1: renamed from KS; footprint (none) -> Button_Switch_Keyboard:SW_Cherry_MX_1.00u_PCB
- KT1: renamed from KT; footprint (none) -> Button_Switch_Keyboard:SW_Cherry_MX_1.00u_PCB
- KU1: renamed from KU; footprint (none) -> Button_Switch_Keyboard:SW_Cherry_MX_1.00u_PCB
- KV1: renamed from KV; footprint (none) -> Button_Switch_Keyboard:SW_Cherry_MX_1.00u_PCB
- KW1: renamed from KW; footprint (none) -> Button_Switch_Keyboard:SW_Cherry_MX_1.00u_PCB
- KX1: renamed from KX; footprint (none) -> Button_Switch_Keyboard:SW_Cherry_MX_1.00u_PCB
- KY1: renamed from KY; footprint (none) -> Button_Switch_Keyboard:SW_Cherry_MX_1.00u_PCB
- KZ1: renamed from KZ; footprint (none) -> Button_Switch_Keyboard:SW_Cherry_MX_1.00u_PCB
- K_Bsc1: renamed from K_Bsc; footprint (none) -> Button_Switch_Keyboard:SW_Cherry_MX_1.50u_PCB
- K_CL1: renamed from K_CL; footprint (none) -> Button_Switch_Keyboard:SW_Cherry_MX_1.75u_PCB
- K_Ent-1: footprint (none) -> Button_Switch_Keyboard:SW_Cherry_MX_ISOEnter_PCB
- K_Ent1: renamed from K_Ent; footprint (none) -> Button_Switch_Keyboard:SW_Cherry_MX_2.25u_PCB
- K_Esc1: renamed from K_Esc; footprint (none) -> Button_Switch_Keyboard:SW_Cherry_MX_1.00u_PCB
- K_Fn1: renamed from K_Fn; footprint (none) -> Button_Switch_Keyboard:SW_Cherry_MX_1.25u_PCB
- K_LA1: renamed from K_LA; footprint (none) -> Button_Switch_Keyboard:SW_Cherry_MX_1.25u_PCB
- K_LC1: renamed from K_LC; footprint (none) -> Button_Switch_Keyboard:SW_Cherry_MX_1.25u_PCB
- K_LS-1: footprint (none) -> Button_Switch_Keyboard:SW_Cherry_MX_1.25u_PCB
- K_LS1: renamed from K_LS; footprint (none) -> Button_Switch_Keyboard:SW_Cherry_MX_2.25u_PCB
- K_LSu1: renamed from K_LSu; footprint (none) -> Button_Switch_Keyboard:SW_Cherry_MX_1.25u_PCB
- K_Men1: renamed from K_Men; footprint (none) -> Button_Switch_Keyboard:SW_Cherry_MX_1.25u_PCB
- K_RA1: renamed from K_RA; footprint (none) -> Button_Switch_Keyboard:SW_Cherry_MX_1.25u_PCB
- K_RC1: renamed from K_RC; footprint (none) -> Button_Switch_Keyboard:SW_Cherry_MX_1.25u_PCB
- K_RS1: renamed from K_RS; footprint (none) -> Button_Switch_Keyboard:SW_Cherry_MX_2.75u_PCB
- K_SPC1: renamed from K_SPC; footprint (none) -> Button_Switch_Keyboard:SW_Cherry_MX_6.25u_PCB
- K_Tb1: renamed from K_Tb; footprint (none) -> Button_Switch_Keyboard:SW_Cherry_MX_1.50u_PCB
- LED1: renamed from LED; footprint (none) -> LED_THT:LED_D3.0mm
- LED2, LED3, LED4: footprint (none) -> LED_THT:LED_D3.0mm
- R1, R10, R2, R3, R4, R5, R6, R7, R8, R9: footprint (none) -> Resistor_THT:R_Axial_DIN0207_L6.3mm_D2.5mm_P7.62mm_Horizontal
- SW1, SW2: footprint (none) -> Button_Switch_THT:SW_PUSH_6mm
- U1: footprint Package_DIP:DIP-40_W15.24mm -> Package_DIP:DIP-40_W15.24mm_Socket
- Y1: footprint (none) -> Crystal:Crystal_HC49-4H_Vertical
Connections:
- net SCK_R is gone; now on net col_14: U1.14 (PD0)
- net SDA_R is gone; now on net col_13: U1.15 (PD1)
- net +5V: now also J3.4 (Pin_4), J4.4 (Pin_4), J5.4 (Pin_4), J6.4 (Pin_4), R11.1, R12.1, U2.18 (~RESET~), U2.9 (VDD), U3.18 (~RESET~), U3.9 (VDD), U4.18 (~RESET~), U4.9 (VDD)
- net GND: now also U1.11 (GND), U1.31 (GND), J2.1 (Pin_1), J3.1 (Pin_1), J4.1 (Pin_1), J5.1 (Pin_1), J6.1 (Pin_1), LED5.1 (K), LED6.1 (K), LED7.1 (K), U2.10 (VSS), U2.15 (A0), U3.10 (VSS), U3.16 (A1), U4.10 (VSS), U4.15 (A0), U4.16 (A1)
- net VCC: now also J2.8 (Pin_8)
- net col_13: no longer U1.23 (PC1)
- net col_14: no longer U1.22 (PC0)
- net col_f0: now also U2.3 (GPB2)
- net col_f1: now also U2.4 (GPB3)
- net col_f10: now also U2.25 (GPA4)
- net col_f11: now also U2.26 (GPA5)
- net col_f2: now also U2.5 (GPB4)
- net col_f3: now also U2.6 (GPB5)
- net col_f4: now also U2.7 (GPB6)
- net col_f5: now also U2.8 (GPB7)
- net col_f6: now also U2.21 (GPA0)
- net col_f7: now also U2.22 (GPA1)
- net col_f8: now also U2.23 (GPA2)
- net col_f9: now also U2.24 (GPA3)
- net col_l1: now also U3.4 (GPB3), U3.6 (GPB5)
- net col_l2: now also U3.7 (GPB6)
- net col_l3: now also U3.8 (GPB7)
- net col_r1: now also U4.6 (GPB5)
- net col_r2: now also U4.7 (GPB6)
- net col_r3: now also U4.8 (GPB7)
- net col_r4: now also U4.21 (GPA0)
- net row_f0: now also U2.1 (GPB0)
- net row_f1: now also U2.2 (GPB1)
- net row_l1: now also U3.1 (GPB0)
- net row_l2: now also U3.2 (GPB1)
- net row_l3: now also U3.3 (GPB2)
- net row_l5: now also U3.5 (GPB4)
- net row_r1: now also U4.1 (GPB0)
- net row_r2: now also U4.2 (GPB1)
- net row_r3: now also U4.3 (GPB2)
- net row_r4: now also U4.4 (GPB3)
- net row_r5: now also U4.5 (GPB4)
- net at R6.2: now also J2.4 (Pin_4)
- net at DZ3.1 (K), R4.2: now also J2.6 (Pin_6)
- net at DZ2.1 (K), R3.2, R5.2: now also J2.7 (Pin_7)
- net at R7.2: now also J2.3 (Pin_3)
- net SCK_F renamed CPS_LCK
- net CPS_LCK: now also LED7.2 (A)
- net SCK_L: no longer names the net of U1.33 (PA7)
- net SDA_F: no longer names the net of U1.34 (PA6)
- net SDA_L: no longer names the net of U1.29 (PC7)
- new net NUM_LCK: LED5.2 (A), U4.22 (GPA1)
- new net SCL: J3.3 (Pin_3), J4.3 (Pin_3), J5.3 (Pin_3), J6.3 (Pin_3), R12.2, U1.22 (PC0), U2.12 (SCK), U3.12 (SCK), U4.12 (SCK)
- new net SCR_LCK: LED6.2 (A), U3.21 (GPA0)
- new net SDA: J3.2 (Pin_2), J4.2 (Pin_2), J5.2 (Pin_2), J6.2 (Pin_2), R11.2, U1.23 (PC1), U2.13 (SDA), U3.13 (SDA), U4.13 (SDA)
- no-connect marks 39 -> 33
Other:
- moved on the sheet: C3, C4, C5, DZ2, DZ3, F1, R3, R4, R5, R6, R7

Commit message: Started working on PCB
Parts:
- C1: footprint (none) -> Capacitor_THT:C_Disc_D3.4mm_W2.1mm_P2.50mm
- C2, C4, C5: footprint (none) -> Capacitor_THT:C_Disc_D3.8mm_W2.6mm_P2.50mm
- F1: footprint (none) -> Capacitor_THT:C_Disc_D9.0mm_W5.0mm_P10.00mm
- J1: footprint Connector_PinHeader_1.00mm:PinHeader_2x03_P1.00mm_Vertical -> Connector_PinHeader_2.54mm:PinHeader_2x03_P2.54mm_Vertical
- J2: footprint Connector_PinHeader_1.00mm:PinHeader_1x08_P1.00mm_Vertical -> Connector_PinHeader_2.54mm:PinHeader_1x08_P2.54mm_Vertical
- J3, J4, J5, J6: footprint Connector_PinHeader_1.00mm:PinHeader_1x04_P1.00mm_Vertical -> Connector_PinHeader_2.54mm:PinHeader_1x04_P2.54mm_Vertical
- K_L10, K_L11, K_L12, K_L13, K_L14, K_L15, K_L16, K_L4, K_L5, K_L6, K_L7, K_L8, K_L9, K_R1, K_R10, K_R11, K_R12, K_R13, K_R14, K_R16-1, K_R17, K_R18, K_R2, K_R3, K_R4, K_R5, K_R6, K_R7, K_R9: footprint (none) -> Button_Switch_Keyboard:SW_Cherry_MX_1.00u_PCB
- K_R15, K_R8: footprint (none) -> Button_Switch_Keyboard:SW_Cherry_MX_2.00u_Vertical_PCB
- K_R16: footprint (none) -> Button_Switch_Keyboard:SW_Cherry_MX_2.00u_PCB

Commit message: Routing p.1
Parts:
- added D_L10, D_L12, D_R12, D_R20, D_RS2: D, Diode_THT:D_DO-35_SOD27_P7.62mm_Horizontal, symbol Device:D
- added J10, J4, J6, J8: I2C, Connector_PinHeader_2.54mm:PinHeader_1x04_P2.54mm_Vertical, symbol Connector:Conn_01x04_Female
- added K_Fn1-1.5u1, K_LA2-1.5u1, K_LC2-1.5u1, K_RC2-1.5u1, K_RS1-1.5u1, K_RS2: KEYSW, Button_Switch_Keyboard:SW_Cherry_MX_1.50u_PCB, symbol keyboard_parts:KEYSW
- added K_L10, K_L12, K_LSu2-1u1, K_Men1-1u1, K_R12, K_R16-1, K_R20, K_R8-1: KEYSW, Button_Switch_Keyboard:SW_Cherry_MX_1.00u_PCB, symbol keyboard_parts:KEYSW
- added K_RS1-1.25u1, K_RS2-1.25u1: KEYSW, Button_Switch_Keyboard:SW_Cherry_MX_1.25u_PCB, symbol keyboard_parts:KEYSW
- added K_SPC2-7u1: KEYSW, MX_Only:MXOnly-7U-NoLED, symbol keyboard_parts:KEYSW
- added R_CPS1, R_NUM1, R_SCR1: 1.5k, Resistor_THT:R_Axial_DIN0207_L6.3mm_D2.5mm_P7.62mm_Horizontal, symbol Device:R
- renumbered D_L4 to D_L1, D_L13 to D_L11, D_L14 to D_L13, D_L15 to D_L14, D_L16 to D_L15, D_L5 to D_L2, D_L6 to D_L3, D_L7 to D_L4, D_L8 to D_L5, D_L9 to D_L6, D_L10 to D_L7, D_L11 to D_L8, D_L12 to D_L9, D_R12 to D_R13, D_R13 to D_R14, D_R14 to D_R15, D_R15 to D_R16, D_R16 to D_R17, D_R17 to D_R18, D_R18 to D_R19, J4 to J5, J5 to J7, J6 to J9, K_L4 to K_L1, K_L13 to K_L11, K_L14 to K_L13, K_L15 to K_L14, K_L16 to K_L15, K_L5 to K_L2, K_L6 to K_L3, K_L7 to K_L4, K_L8 to K_L5, K_L9 to K_L6, K_L10 to K_L7, K_L11 to K_L8, K_L12 to K_L9, K_R12 to K_R13, K_R13 to K_R14, K_R14 to K_R15, K_R15 to K_R16, K_R16 to K_R17, K_R16-1 to K_R17-1, K_R17 to K_R18, K_R18 to K_R19
Connections:
- net +5V: now also C6.1, C7.1, C8.1, J10.4 (Pin_4), J4.4 (Pin_4), J6.4 (Pin_4), J8.4 (Pin_4)
- net GND: now also J10.1 (Pin_1), J4.1 (Pin_1), J6.1 (Pin_1), J8.1 (Pin_1), R_CPS1.1, R_NUM1.1, R_SCR1.1; no longer LED5.1 (K), LED6.1 (K), LED7.1 (K)
- net SCL: now also J10.3 (Pin_3), J4.3 (Pin_3), J6.3 (Pin_3), J8.3 (Pin_3)
- net SCR_LCK: now also U3.1 (GPB0); no longer U3.21 (GPA0)
- net SDA: now also J10.2 (Pin_2), J4.2 (Pin_2), J6.2 (Pin_2), J8.2 (Pin_2)
- net VCC: no longer C6.1, C7.1, C8.1
- net col_1: now also K_LC2-1.5u1.1
- net col_13: now also K_Fn1-1.5u1.1
- net col_14: now also K_RS1.1, K_Men1-1u1.1, K_RS1-1.25u1.1, K_RS1-1.5u1.1
- net col_15: now also K_RC2-1.5u1.1, K_RS2-1.25u1.1, K_RS2.1; no longer K_RS1.1
- net col_2: now also K_LSu2-1u1.1
- net col_3: now also K_LA2-1.5u1.1
- net col_8: now also K_SPC2-7u1.1
- net col_f0: now also U2.8 (GPB7); no longer U2.3 (GPB2)
- net col_f1: now also U2.7 (GPB6); no longer U2.4 (GPB3)
- net col_f10: now also U2.22 (GPA1); no longer U2.25 (GPA4)
- net col_f11: now also U2.21 (GPA0); no longer U2.26 (GPA5)
- net col_f2: now also U2.6 (GPB5); no longer U2.5 (GPB4)
- net col_f3: now also U2.5 (GPB4); no longer U2.6 (GPB5)
- net col_f4: now also U2.4 (GPB3); no longer U2.7 (GPB6)
- net col_f5: now also U2.3 (GPB2); no longer U2.8 (GPB7)
- net col_f6: now also U2.26 (GPA5); no longer U2.21 (GPA0)
- net col_f7: now also U2.25 (GPA4); no longer U2.22 (GPA1)
- net col_f8: now also U2.24 (GPA3); no longer U2.23 (GPA2)
- net col_f9: now also U2.23 (GPA2); no longer U2.24 (GPA3)
- net col_l1: now also U3.25 (GPA4), K_L10.1; no longer D_L11.1 (K), U3.4 (GPB3), U3.6 (GPB5)
- net col_l2: now also U3.26 (GPA5); no longer U3.7 (GPB6)
- net col_l3: now also U3.27 (GPA6), K_L12.1; no longer U3.8 (GPB7)
- net col_r4: now also K_R12.1, K_R16-1.1, K_R20.1, K_R8-1.1
- net row_l1: now also U3.21 (GPA0); no longer U3.1 (GPB0)
- net row_l2: now also U3.22 (GPA1); no longer U3.2 (GPB1)
- net row_l3: now also U3.23 (GPA2); no longer U3.3 (GPB2)
- net row_l5: now also U3.28 (GPA7); no longer U3.5 (GPB4)
- net row_r3: now also D_R12.1 (K)
- net row_r5: now also D_R20.1 (K)
- net at D_LC1.2 (A), K_LC1.2: now also K_LC2-1.5u1.2
- net at D_LSu1.2 (A), K_LSu1.2: now also K_LSu2-1u1.2
- net at D_LA1.2 (A), K_LA1.2: now also K_LA2-1.5u1.2
- net at D_SPC1.2 (A), K_SPC1.2: now also K_SPC2-7u1.2
- net at D_R8.2 (A), K_R8.2: now also K_R8-1.2
- net at D_R16.2 (A), K_R16.2: now also K_R16-1.2
- net at D_Fn1.2 (A), K_Fn1.2: now also K_Fn1-1.5u1.2
- net at D_Men1.2 (A), K_Men1.2: now also K_Men1-1u1.2
- net at D_RS1.2 (A), K_RS1.2: now also K_RS1-1.25u1.2, K_RS1-1.5u1.2
- net at D_RC1.2 (A), K_RC1.2: now also K_RC2-1.5u1.2
- net row_l4: now reaches U3.24 (GPA3)
- net row_l4: now also D_L11.1 (K), D_L10.1 (K), D_L12.1 (K)
- new net: D_L10.2 (A), K_L10.2
- new net: LED7.1 (K), R_CPS1.2
- new net: D_L12.2 (A), K_L12.2
- new net: LED5.1 (K), R_NUM1.2
- new net: LED6.1 (K), R_SCR1.2
- new net: D_R12.2 (A), K_R12.2
- new net: D_R20.2 (A), K_R20.2
- new net: D_RS2.2 (A), K_RS2-1.25u1.2, K_RS2.2
- no-connect marks 33 -> 32
Other:
- moved on the sheet: J3, J5, J7, J9
