File: svarog-keyboard.kicad_pcb (KiCad board)
At the start: 2 copper layers, 285 parts, among them J1 AVR-ISP-6, J2 Conn_01x08_Male, J3 I2C, J4 I2C, J5 I2C, J6 I2C, K1 KEYSW, K10 KEYSW, K11 KEYSW, K12 KEYSW, K13 KEYSW, K13-1 KEYSW, K14 KEYSW, K14-1 KEYSW, K14-2 KEYSW, K15 KEYSW, K16 KEYSW, K17 KEYSW, K18 KEYSW, K19 KEYSW, K2 KEYSW, K20 KEYSW, K21 KEYSW, K3 KEYSW, K4 KEYSW, K5 KEYSW, K6 KEYSW, K7 KEYSW, K8 KEYSW, K9 KEYSW, SW1 SW_BOOT, SW2 SW_RESET, U1 ATmega32A-PU, U2 MCP23017_SP, U3 MCP23017_SP, U4 MCP23017_SP, Y1 Crystal

Commit message: Routing p.1
Parts:
- removed D_L16: D, Diode_THT:D_DO-35_SOD27_P7.62mm_Horizontal
- removed K_L16: KEYSW, Button_Switch_Keyboard:SW_Cherry_MX_1.00u_PCB
- added D_L1: D, Diode_THT:D_DO-35_SOD27_P7.62mm_Horizontal, F.Cu at (39.6, 162.6)
- added D_L2: D, Diode_THT:D_DO-35_SOD27_P7.62mm_Horizontal, F.Cu at (59.7, 162.6)
- added D_L3: D, Diode_THT:D_DO-35_SOD27_P7.62mm_Horizontal, F.Cu at (80.0, 162.6)
- added D_R19: D, Diode_THT:D_DO-35_SOD27_P7.62mm_Horizontal, F.Cu at (590.3, 214.6)
- added D_R20: D, Diode_THT:D_DO-35_SOD27_P7.62mm_Horizontal, F.Cu at (596.3, 200.7)
- added D_RS2: D, Diode_THT:D_DO-35_SOD27_P7.62mm_Horizontal, F.Cu at (301.2, 119.9)
- added J10: I2C, Connector_PinHeader_2.54mm:PinHeader_1x04_P2.54mm_Vertical, F.Cu at (442.0, 153.2)
- added J4: I2C, Connector_PinHeader_2.54mm:PinHeader_1x04_P2.54mm_Vertical, F.Cu at (424.2, 153.7)
- added J8: I2C, Connector_PinHeader_2.54mm:PinHeader_1x04_P2.54mm_Vertical, F.Cu at (101.6, 154.2)
- added J9: I2C, Connector_PinHeader_2.54mm:PinHeader_1x04_P2.54mm_Vertical, F.Cu at (530.4, 153.7)
- added K_Fn1-1.5u1: KEYSW, Button_Switch_Keyboard:SW_Cherry_MX_1.50u_PCB, F.Cu at (358.1, 233.7)
- added K_L1: KEYSW, Button_Switch_Keyboard:SW_Cherry_MX_1.00u_PCB, F.Cu at (52.1, 152.4)
- added K_L2: KEYSW, Button_Switch_Keyboard:SW_Cherry_MX_1.00u_PCB, F.Cu at (72.4, 152.4)
- added K_L3: KEYSW, Button_Switch_Keyboard:SW_Cherry_MX_1.00u_PCB, F.Cu at (92.7, 152.4)
- added K_LA2-1.5u1: KEYSW, Button_Switch_Keyboard:SW_Cherry_MX_1.50u_PCB, F.Cu at (193.0, 233.7)
- added K_LC2-1.5u1: KEYSW, Button_Switch_Keyboard:SW_Cherry_MX_1.50u_PCB, F.Cu at (142.2, 233.7)
- added K_LSu2-1u1: KEYSW, Button_Switch_Keyboard:SW_Cherry_MX_1.00u_PCB, F.Cu at (167.6, 233.7)
- added K_Men1-1u1: KEYSW, Button_Switch_Keyboard:SW_Cherry_MX_1.00u_PCB, F.Cu at (383.5, 233.7)
- added K_R17-1: KEYSW, Button_Switch_Keyboard:SW_Cherry_MX_1.00u_PCB, F.Cu at (458.5, 233.7)
- added K_R19: KEYSW, Button_Switch_Keyboard:SW_Cherry_MX_1.00u_PCB, F.Cu at (499.1, 233.7)
- added K_R20: KEYSW, Button_Switch_Keyboard:SW_Cherry_MX_1.00u_PCB, F.Cu at (519.4, 233.7)
- added K_R8-1: KEYSW, Button_Switch_Keyboard:SW_Cherry_MX_1.00u_PCB, F.Cu at (519.4, 172.7)
- added K_RC2-1.5u1: KEYSW, Button_Switch_Keyboard:SW_Cherry_MX_1.50u_PCB, F.Cu at (408.9, 233.7)
- added K_RS1-1.25u1: KEYSW, Button_Switch_Keyboard:SW_Cherry_MX_1.25u_PCB, F.Cu at (384.8, 213.4)
- added K_RS1-1.5u1: KEYSW, Button_Switch_Keyboard:SW_Cherry_MX_1.50u_PCB, F.Cu at (387.4, 213.4)
- added K_RS2: KEYSW, Button_Switch_Keyboard:SW_Cherry_MX_1.50u_PCB, F.Cu at (411.5, 213.4)
- added K_RS2-1.25u1: KEYSW, Button_Switch_Keyboard:SW_Cherry_MX_1.25u_PCB, F.Cu at (414.0, 213.4)
- added K_SPC2-7u1: KEYSW, MX_Only:MXOnly-7U-NoLED, F.Cu at (273.1, 238.8)
- added R_CPS1: 1.5k, Resistor_THT:R_Axial_DIN0207_L6.3mm_D2.5mm_P7.62mm_Horizontal, F.Cu at (353.6, 100.8)
- added R_NUM1: 1.5k, Resistor_THT:R_Axial_DIN0207_L6.3mm_D2.5mm_P7.62mm_Horizontal, F.Cu at (461.5, 144.8)
- added R_SCR1: 1.5k, Resistor_THT:R_Axial_DIN0207_L6.3mm_D2.5mm_P7.62mm_Horizontal, F.Cu at (95.8, 137.2)
- K_R15: footprint Button_Switch_Keyboard:SW_Cherry_MX_2.00u_Vertical_PCB -> Button_Switch_Keyboard:SW_Cherry_MX_1.00u_PCB
- K_R16: footprint Button_Switch_Keyboard:SW_Cherry_MX_2.00u_PCB -> Button_Switch_Keyboard:SW_Cherry_MX_2.00u_Vertical_PCB
- K_R17: footprint Button_Switch_Keyboard:SW_Cherry_MX_1.00u_PCB -> Button_Switch_Keyboard:SW_Cherry_MX_2.00u_PCB
- moved D_R12 543.6 mm to (585.0, 151.8)
- moved D_R2 543.6 mm to (585.0, 155.4)
- moved D_R6 543.6 mm to (560.9, 175.6)
- moved D_R7 543.6 mm to (560.9, 172.0)
- moved D_R10 426.4 mm to (581.6, 184.0)
- moved D_R5 426.4 mm to (581.6, 191.1)
- moved D_R9 426.4 mm to (581.6, 187.6)
- moved C7 408.7 mm to (507.7, 142.2), turned to 90 degrees
- moved D_F22 405.8 mm to (361.9, 58.4), turned to 90 degrees
- moved D_F23 394.9 mm to (382.3, 58.4), turned to 90 degrees
- moved D1 393.0 mm to (140.0, 113.0), turned to 270 degrees
- moved D14-2 385.0 mm to (148.3, 119.9), turned to 270 degrees
- moved D_F12 366.5 mm to (402.6, 78.7), turned to 90 degrees
- moved C5 363.8 mm to (404.7, 106.4)
- moved DR1 356.1 mm to (181.6, 115.3), turned to 270 degrees
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- renumbered J4 to J5, J5 to J7
Connections:
- C6 pad 1: VCC -> +5V
- C7 pad 1: VCC -> +5V
- C8 pad 1: VCC -> +5V
- D_L10 pad 1: row_l3 -> row_l4
- D_L11 pad 1: row_l3 -> row_l4
- D_L12 pad 1: row_l3 -> row_l4
- D_L13 pad 1: col_l1 -> row_l5
- D_L4 pad 1: row_l1 -> row_l2
- D_L5 pad 1: row_l1 -> row_l2
- D_L6 pad 1: row_l1 -> row_l2
- D_L7 pad 1: row_l2 -> row_l3
- D_L8 pad 1: row_l2 -> row_l3
- D_L9 pad 1: row_l2 -> row_l3
- D_R12 pad 1: row_r4 -> row_r3
- D_R16 pad 1: row_r5 -> row_r4
- J2 pad 2: Net-(J2-Pad2) -> (no net)
- J2 pad 5: Net-(J2-Pad5) -> (no net)
- K_L13 pad 1: col_l2 -> col_l1
- K_L14 pad 1: col_l1 -> col_l2
- K_L15 pad 1: col_l2 -> col_l3
- K_R12 pad 1: col_r1 -> col_r4
- K_R13 pad 1: col_r2 -> col_r1
- K_R14 pad 1: col_r3 -> col_r2
- K_R15 pad 1: col_r4 -> col_r3
- K_R16 pad 1: col_r1 -> col_r4
- K_R16-1 pad 1: col_r1 -> col_r4
- K_R17 pad 1: col_r2 -> col_r1
- K_R18 pad 1: col_r3 -> col_r2
- K_RS1 pad 1: col_15 -> col_14
- LED5 pad 1: GND -> Net-(LED5-Pad1)
- LED6 pad 1: GND -> Net-(LED6-Pad1)
- LED7 pad 1: GND -> Net-(LED7-Pad1)
- U1 pad 29: Net-(U1-Pad29) -> (no net)
- U1 pad 32: Net-(U1-Pad32) -> (no net)
- U1 pad 33: Net-(U1-Pad33) -> (no net)
- U1 pad 34: Net-(U1-Pad34) -> (no net)
- U2 pad 11: Net-(U2-Pad11) -> (no net)
- U2 pad 14: Net-(U2-Pad14) -> (no net)
- U2 pad 16: Net-(U2-Pad16) -> (no net)
- U2 pad 17: Net-(U2-Pad17) -> (no net)
- U2 pad 19: Net-(U2-Pad19) -> (no net)
- U2 pad 20: Net-(U2-Pad20) -> (no net)
- U2 pad 21: col_f6 -> col_f11
- U2 pad 22: col_f7 -> col_f10
- U2 pad 23: col_f8 -> col_f9
- U2 pad 24: col_f9 -> col_f8
- U2 pad 25: col_f10 -> col_f7
- U2 pad 26: col_f11 -> col_f6
- U2 pad 27: Net-(U2-Pad27) -> (no net)
- U2 pad 28: Net-(U2-Pad28) -> (no net)
- U2 pad 3: col_f0 -> col_f5
- U2 pad 4: col_f1 -> col_f4
- U2 pad 5: col_f2 -> col_f3
- U2 pad 6: col_f3 -> col_f2
- U2 pad 7: col_f4 -> col_f1
- U2 pad 8: col_f5 -> col_f0
- U3 pad 1: row_l1 -> SCR_LCK
- U3 pad 11: Net-(U3-Pad11) -> (no net)
- U3 pad 14: Net-(U3-Pad14) -> (no net)
- U3 pad 15: Net-(U3-Pad15) -> (no net)
- U3 pad 17: Net-(U3-Pad17) -> (no net)
- U3 pad 19: Net-(U3-Pad19) -> (no net)
- U3 pad 2: row_l2 -> (no net)
- U3 pad 20: Net-(U3-Pad20) -> (no net)
- U3 pad 21: SCR_LCK -> row_l1
- U3 pad 22: Net-(U3-Pad22) -> row_l2
- U3 pad 23: Net-(U3-Pad23) -> row_l3
- U3 pad 24: Net-(U3-Pad24) -> row_l4
- U3 pad 25: Net-(U3-Pad25) -> col_l1
- U3 pad 26: Net-(U3-Pad26) -> col_l2
- U3 pad 27: Net-(U3-Pad27) -> col_l3
- U3 pad 28: Net-(U3-Pad28) -> row_l5
- U3 pad 3: row_l3 -> (no net)
- U3 pad 4: col_l1 -> (no net)
- U3 pad 5: row_l5 -> (no net)
- U3 pad 6: col_l1 -> (no net)
- U3 pad 7: col_l2 -> (no net)
- U3 pad 8: col_l3 -> (no net)
- U4 pad 11: Net-(U4-Pad11) -> (no net)
- U4 pad 14: Net-(U4-Pad14) -> (no net)
- U4 pad 17: Net-(U4-Pad17) -> (no net)
- U4 pad 19: Net-(U4-Pad19) -> (no net)
- U4 pad 20: Net-(U4-Pad20) -> (no net)
- U4 pad 23: Net-(U4-Pad23) -> (no net)
- U4 pad 24: Net-(U4-Pad24) -> (no net)
- U4 pad 25: Net-(U4-Pad25) -> (no net)
- U4 pad 26: Net-(U4-Pad26) -> (no net)
- U4 pad 27: Net-(U4-Pad27) -> (no net)
- U4 pad 28: Net-(U4-Pad28) -> (no net)
Routing:
- net row_l5: track 0.00 -> 142.9 mm
- net row_l4: track 0.00 -> 121.6 mm
- net col_l1: track 0.00 -> 114.3 mm
- net row_l3: track 0.00 -> 101.9 mm
- net col_l2: track 0.00 -> 97.6 mm
- net col_l3: track 0.00 -> 95.3 mm
- net +5V: track 0.00 -> 92.0 mm
- net SDA: track 0.00 -> 90.4 mm
- net SCL: track 0.00 -> 87.9 mm
- net row_l2: track 0.00 -> 82.3 mm
- net row_l1: track 0.00 -> 65.2 mm
- net Net-(LED3-Pad1): track 0.00 -> 8.42 mm
- net Net-(LED6-Pad1): track 0.00 -> 7.61 mm
- net Net-(D_L8-Pad2): track 0.00 -> 6.35 mm
- net Net-(D_L5-Pad2): track 0.00 -> 6.35 mm
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
Commit message: Removed Traces, cleanup
Parts:
- removed C6, C7, C8: 4.7u, Capacitor_THT:CP_Radial_D4.0mm_P1.50mm
- moved D_R1 198.7 mm to (418.6, 163.3), turned to 90 degrees
- moved D_R17 189.6 mm to (418.6, 239.5), turned to 90 degrees
- moved D_R18 167.9 mm to (456.4, 243.8)
- moved D_R9 163.6 mm to (418.6, 201.4), turned to 90 degrees
- moved D_R5 163.3 mm to (418.6, 182.4), turned to 90 degrees
- moved D_R13 154.9 mm to (418.6, 220.5), turned to 90 degrees
- moved D_R3 149.9 mm to (456.7, 163.3), turned to 90 degrees
- moved D_R2 147.6 mm to (437.6, 163.3), turned to 90 degrees
- moved D_R10 145.0 mm to (437.6, 201.4), turned to 90 degrees
- moved D_R4 141.7 mm to (475.7, 163.3), turned to 90 degrees
- moved D_R16 139.5 mm to (468.1, 224.8)
- moved D_R19 135.9 mm to (456.7, 239.5), turned to 90 degrees
- moved D_R20 135.2 mm to (468.1, 243.8)
- moved D_R15 133.1 mm to (456.7, 220.5), turned to 90 degrees
- moved D_R12 128.7 mm to (468.1, 205.7)
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Routing:
- net row_l5: track 142.9 -> 0.00 mm
- net row_l4: track 121.6 -> 0.00 mm
- net col_l1: track 114.3 -> 0.00 mm
- net row_l3: track 101.9 -> 0.00 mm
- net col_l2: track 97.6 -> 0.00 mm
- net col_l3: track 95.3 -> 0.00 mm
- net row_l2: track 82.3 -> 0.00 mm
- net SDA: track 90.4 -> 14.1 mm
- net SCL: track 87.9 -> 14.8 mm
- net +5V: track 92.0 -> 21.7 mm
- net row_l1: track 65.2 -> 0.00 mm
- net Net-(LED3-Pad1): track 8.42 -> 0.00 mm
- net Net-(LED6-Pad1): track 7.61 -> 0.00 mm
- net Net-(D_L8-Pad2): track 6.35 -> 0.00 mm
- net Net-(D_L5-Pad2): track 6.35 -> 0.00 mm
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
Commit message: Wired [TODO] main matrix and [FULL] side matrixes
Parts:
- removed K_RS1-1.25u1: KEYSW, Button_Switch_Keyboard:SW_Cherry_MX_1.25u_PCB
- added K_RS1-1.75u1: KEYSW, Button_Switch_Keyboard:SW_Cherry_MX_1.75u_PCB, F.Cu at (374.1, 210.3)
- K_RS1-1u1: renamed from K_RS1-1.5u1; footprint Button_Switch_Keyboard:SW_Cherry_MX_1.50u_PCB -> Button_Switch_Keyboard:SW_Cherry_MX_1.00u_PCB
- K_RS2: footprint Button_Switch_Keyboard:SW_Cherry_MX_1.50u_PCB -> Button_Switch_Keyboard:SW_Cherry_MX_1.00u_PCB
- K_RS2-1.75u1: renamed from K_RS2-1.25u1; footprint Button_Switch_Keyboard:SW_Cherry_MX_1.25u_PCB -> Button_Switch_Keyboard:SW_Cherry_MX_1.75u_PCB
- moved D_RC1 141.6 mm to (383.3, 239.5), turned to 90 degrees
- moved D_Men1 138.4 mm to (359.7, 239.5), turned to 90 degrees
- moved D_Fn1 134.4 mm to (335.8, 239.5), turned to 90 degrees
- moved D_RA1 125.1 mm to (314.2, 239.5), turned to 90 degrees
- moved D_RS1 123.1 mm to (354.8, 220.5), turned to 90 degrees
- moved D21 121.5 mm to (336.0, 220.5), turned to 90 degrees
- moved D_SPC1 118.8 mm to (242.3, 239.5), turned to 90 degrees
- moved D_LC1 118.4 mm to (121.7, 239.5), turned to 90 degrees
- moved D14-1 117.5 mm to (364.5, 201.4), turned to 90 degrees
- moved D_LSu1 117.5 mm to (145.5, 239.5), turned to 90 degrees
- moved D_LA1 117.4 mm to (169.4, 239.5), turned to 90 degrees
- moved D20 117.0 mm to (316.7, 220.5), turned to 90 degrees
- moved D_RS2 116.9 mm to (352.8, 224.8), turned to 0 degrees
- moved D18 116.1 mm to (345.4, 201.4), turned to 90 degrees
- moved D19 113.1 mm to (297.7, 220.5), turned to 90 degrees
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Connections:
- D_RS2 pad 1: (no net) -> row_4
- U1 pad 1: row_5 -> col_1
- U1 pad 2: row_3 -> col_3
- U1 pad 3: row_1 -> col_5
- U1 pad 36: col_5 -> row_1
- U1 pad 37: col_3 -> row_2
- U1 pad 38: col_1 -> row_3
- U1 pad 39: row_2 -> row_4
- U1 pad 40: row_4 -> row_5
- U4 pad 1: row_r1 -> NUM_LCK
- U4 pad 2: row_r2 -> (no net)
- U4 pad 21: col_r4 -> row_r1
- U4 pad 22: NUM_LCK -> (no net)
- U4 pad 25: (no net) -> row_r2
- U4 pad 26: (no net) -> row_r3
- U4 pad 27: (no net) -> row_r4
- U4 pad 28: (no net) -> row_r5
- U4 pad 3: row_r3 -> (no net)
- U4 pad 4: row_r4 -> (no net)
- U4 pad 5: row_r5 -> col_r4
- U4 pad 6: col_r1 -> col_r3
- U4 pad 8: col_r3 -> col_r1
Routing:
- net +5V: track 21.7 -> 644.2 mm, vias 0 -> 2
- net SCL: track 14.8 -> 543.0 mm, vias 0 -> 4
- net SDA: track 14.1 -> 528.8 mm, vias 0 -> 4
- net row_5: track 0.00 -> 374.8 mm
- net row_4: track 0.00 -> 370.4 mm
- net row_3: track 0.00 -> 350.8 mm
- net row_1: track 0.00 -> 319.0 mm
- net row_2: track 0.00 -> 311.2 mm
- net row_r5: track 0.00 -> 159.6 mm
- net row_l5: track 0.00 -> 135.9 mm, vias 0 -> 1
- net row_r4: track 0.00 -> 135.7 mm, vias 0 -> 1
- net row_l4: track 0.00 -> 119.3 mm, vias 0 -> 1
- net col_r1: track 0.00 -> 118.4 mm
- net col_14: track 0.00 -> 116.7 mm
- net row_r3: track 0.00 -> 116.3 mm, vias 0 -> 1
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
Commit message: Rev 0.1 [ALPHA] [UNTESTED]
Parts:
- added  : , keyboard_parts:HOLE_M3, F.Cu at (417.2, 246.5)
- added  : , keyboard_parts:HOLE_M3, F.Cu at (491.5, 141.2)
- added  : , keyboard_parts:HOLE_M3, F.Cu at (456.4, 187.7)
- added  : , keyboard_parts:HOLE_M3, F.Cu at (437.6, 206.0)
- added  : , keyboard_parts:HOLE_M3, F.Cu at (485.4, 242.1)
- added  : , keyboard_parts:HOLE_M3, F.Cu at (245.1, 170.2)
- added  : , keyboard_parts:HOLE_M3, F.Cu at (406.4, 226.8)
- added  : , keyboard_parts:HOLE_M3, F.Cu at (160.8, 141.0)
- added  : , keyboard_parts:HOLE_M3, F.Cu at (124.5, 170.4)
- added  : , keyboard_parts:HOLE_M3, F.Cu at (324.6, 137.7)
- added  : , keyboard_parts:HOLE_M3, F.Cu at (230.9, 205.5)
- added  : , keyboard_parts:HOLE_M3, F.Cu at (51.3, 243.1)
- added  : , keyboard_parts:HOLE_M3, F.Cu at (286.8, 233.4)
- added  : , keyboard_parts:HOLE_M3, F.Cu at (283.2, 300.0)
- added  : , keyboard_parts:HOLE_M3, F.Cu at (369.3, 271.3)
- added  : , keyboard_parts:HOLE_M3, F.Cu at (255.1, 251.5)
- added  : , keyboard_parts:HOLE_M3, F.Cu at (293.1, 271.3)
- added  : , keyboard_parts:HOLE_M3, F.Cu at (216.9, 271.3)
- added  : , keyboard_parts:HOLE_M3, F.Cu at (140.5, 271.3)
- added  : , keyboard_parts:HOLE_M3, F.Cu at (107.3, 246.4)
- added  : , keyboard_parts:HOLE_M3, F.Cu at (72.9, 206.5)
- added  : , keyboard_parts:HOLE_M3, F.Cu at (51.8, 146.8)
- added  : , keyboard_parts:HOLE_M3, F.Cu at (111.8, 138.4)
- added  : , keyboard_parts:HOLE_M3, F.Cu at (221.7, 235.7)
- added  : , keyboard_parts:HOLE_M3, F.Cu at (124.2, 244.1)
- added  : , keyboard_parts:HOLE_M3, F.Cu at (422.4, 141.5)
- added J11: I2C, Connector_PinHeader_2.54mm:PinHeader_1x04_P2.54mm_Vertical, F.Cu at (209.0, 138.4)
- moved R8 235.8 mm to (228.6, 299.5)
- moved LED2 232.7 mm to (231.4, 298.4)
- moved U2 231.9 mm to (271.5, 292.9), turned to 270 degrees
- moved K_F24 214.9 mm to (362.2, 256.5)
- moved J6 214.8 mm to (359.4, 292.1)
- moved D_F24 214.8 mm to (350.3, 266.7)
- moved K_F23 214.6 mm to (343.2, 256.5)
- moved D_F23 214.4 mm to (331.2, 266.7)
- moved J5 214.4 mm to (158.0, 292.1)
- moved K_F22 214.3 mm to (324.1, 256.5)
- moved D_F22 214.1 mm to (312.2, 266.7)
- moved K_F21 214.0 mm to (305.1, 256.5)
- moved D_F21 213.9 mm to (293.1, 266.7)
- moved K_F20 213.7 mm to (286.0, 256.5)
- moved K_F12 213.7 mm to (362.2, 275.6)
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Connections:
- J2 pad 2: (no net) -> Net-(J2-Pad2)
- J2 pad 5: (no net) -> Net-(J2-Pad5)
- J5 pad 2: SDA -> SDA_F
- J5 pad 3: SCL -> SCL_F
- J6 pad 2: SDA -> SDA_F
- J6 pad 3: SCL -> SCL_F
- U1 pad 1: col_1 -> CPS_LCK
- U1 pad 14: col_14 -> col_11
- U1 pad 15: col_13 -> col_10
- U1 pad 19: col_6 -> col_7
- U1 pad 2: col_3 -> col_15
- U1 pad 20: col_7 -> col_6
- U1 pad 21: col_15 -> col_1
- U1 pad 24: col_12 -> col_2
- U1 pad 25: col_11 -> col_3
- U1 pad 26: col_10 -> col_4
- U1 pad 27: col_9 -> col_5
- U1 pad 29: (no net) -> Net-(U1-Pad29)
- U1 pad 3: col_5 -> col_14
- U1 pad 32: (no net) -> Net-(U1-Pad32)
- U1 pad 33: (no net) -> Net-(U1-Pad33)
- U1 pad 34: (no net) -> Net-(U1-Pad34)
- U1 pad 35: CPS_LCK -> col_9
- U1 pad 4: col_2 -> col_13
- U1 pad 5: col_4 -> col_12
- U2 pad 11: (no net) -> Net-(U2-Pad11)
- U2 pad 14: (no net) -> Net-(U2-Pad14)
- U2 pad 16: (no net) -> Net-(U2-Pad16)
- U2 pad 17: (no net) -> Net-(U2-Pad17)
- U2 pad 19: (no net) -> Net-(U2-Pad19)
- U2 pad 20: (no net) -> Net-(U2-Pad20)
- U2 pad 21: col_f11 -> col_f6
- U2 pad 22: col_f10 -> col_f7
- U2 pad 23: col_f9 -> col_f8
- U2 pad 24: col_f8 -> col_f9
- U2 pad 25: col_f7 -> col_f10
- U2 pad 26: col_f6 -> col_f11
- U2 pad 27: (no net) -> Net-(U2-Pad27)
- U2 pad 28: (no net) -> Net-(U2-Pad28)
- U3 pad 11: (no net) -> Net-(U3-Pad11)
- U3 pad 14: (no net) -> Net-(U3-Pad14)
- U3 pad 15: (no net) -> Net-(U3-Pad15)
- U3 pad 17: (no net) -> Net-(U3-Pad17)
- U3 pad 19: (no net) -> Net-(U3-Pad19)
- U3 pad 2: (no net) -> Net-(U3-Pad2)
- U3 pad 20: (no net) -> Net-(U3-Pad20)
- U3 pad 3: (no net) -> Net-(U3-Pad3)
- U3 pad 4: (no net) -> Net-(U3-Pad4)
- U3 pad 5: (no net) -> Net-(U3-Pad5)
- U3 pad 6: (no net) -> Net-(U3-Pad6)
- U3 pad 7: (no net) -> Net-(U3-Pad7)
- U3 pad 8: (no net) -> Net-(U3-Pad8)
- U4 pad 11: (no net) -> Net-(U4-Pad11)
- U4 pad 14: (no net) -> Net-(U4-Pad14)
- U4 pad 17: (no net) -> Net-(U4-Pad17)
- U4 pad 19: (no net) -> Net-(U4-Pad19)
- U4 pad 2: (no net) -> Net-(U4-Pad2)
- U4 pad 20: (no net) -> Net-(U4-Pad20)
- U4 pad 22: (no net) -> Net-(U4-Pad22)
- U4 pad 23: (no net) -> Net-(U4-Pad23)
- U4 pad 24: (no net) -> Net-(U4-Pad24)
- U4 pad 3: (no net) -> Net-(U4-Pad3)
- U4 pad 4: (no net) -> Net-(U4-Pad4)
Routing:
- net +5V: track 644.2 -> 1046.4 mm, vias 2 -> 7
- net SDA: track 528.8 -> 882.4 mm, vias 4 -> 6
- net SCL: track 543.0 -> 856.7 mm, vias 4 -> 8
- net row_f1: track 0.00 -> 237.8 mm
- net row_f0: track 0.00 -> 218.0 mm
- net col_f11: track 0.00 -> 137.5 mm, vias 0 -> 1
- net row_1: track 319.0 -> 453.6 mm
- net col_f0: track 0.00 -> 132.7 mm
- net row_2: track 311.2 -> 443.6 mm
- net col_15: track 99.0 -> 230.9 mm
- net row_3: track 350.8 -> 481.3 mm
- net row_5: track 374.8 -> 504.0 mm
- net row_4: track 370.4 -> 498.6 mm
- net col_f10: track 0.00 -> 121.4 mm, vias 0 -> 1
- net col_14: track 116.7 -> 235.9 mm
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Other:
- board outline added: 451.1 x 188.2 mm

Commit message: [PRERELEASE]
Routing:
- added copper zone on B.Cu, net GND
- added copper zone on F.Cu, net GND
Changed lines of the file:
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@@
     (pcbplotparams
       (layerselection 0x010fc_ffffffff)
-      (usegerberextensions false)
+      (usegerberextensions true)
       (usegerberattributes false)
       (usegerberadvancedattributes false)
@@
       (outputformat 1)
       (mirror false)
-      (drillshape 1)
+      (drillshape 0)
       (scaleselection 1)
-      (outputdirectory ""))
+      (outputdirectory "gerber/"))
   )
   (net 0 "")
@@
   (segment (start 285.242 124.714) (end 286.004 123.952) (width 0.25) (layer F.Cu) (net 203))
   (segment (start 283.718 124.714) (end 285.242 124.714) (width 0.25) (layer F.Cu) (net 203))
+  (zone (net 1) (net_name GND) (layer F.Cu) (hatch edge 0.508)
+    (connect_pads (clearance 0.508))
+    (min_thickness 0.254)
+    (fill yes (arc_segments 32) (thermal_gap 0.508) (thermal_bridge_width 0.508))
+    (polygon
+      (pts
+        (xy 14.732 15.748) (xy 568.96 19.431) (xy 565.404 367.792) (xy 19.939 360.68)
+      )
+    )
+  )
+  (zone (net 1) (net_name GND) (layer B.Cu) (hatch edge 0.508)
+    (connect_pads (clearance 0.508))
+    (min_thickness 0.254)
+    (fill yes (arc_segments 32) (thermal_gap 0.508) (thermal_bridge_width 0.508))
+    (polygon
+      (pts
+        (xy 19.939 22.987) (xy 561.848 29.21) (xy 559.181 350.901) (xy 22.606 355.346)
+      )
+    )
+  )
 )

Commit message: [FIXED] unconnected row_f4
Connections:
- U2 pad 12: SCL -> SCL_F
- U2 pad 13: SDA -> SDA_F
Routing:
- net SCL: track 856.7 -> 639.1 mm, vias 8 -> 7
- net SCL_F: track 0.00 -> 217.5 mm, vias 0 -> 1
- net SDA: track 882.4 -> 668.0 mm
- net SDA_F: track 0.00 -> 214.4 mm
- net +5V: track 1046.4 -> 1134.1 mm
- net col_f6: track 0.00 -> 54.0 mm, vias 0 -> 1
- net Net-(D_LC1-Pad2): track 7.98 -> 10.4 mm
- net row_f0: track 218.0 -> 219.0 mm
- net GND: vias 0 -> 10
- net (no net): vias 0 -> 1
Other:
- rule via_min_size: 0.4 -> 0.2
